Commit message: Fix #311: rebuild UR5 / iiwa14 / Panda / YAM / PiPER from manufacturer URDFs
These five prebuilts were built against textbook DH approximations or
older vendored URDF revisions. ``module.solve(T)`` returned q such that
``module.fk(q) ≈ T`` at 1e-15, but ``module.fk`` was the textbook FK,
not the manufacturer URDF's. On real hardware (UR5 has a 135 mm
physical shoulder offset that classical DH idealizes away), the EE
landed cm-scale off target.

Per-arm:

- UR5: classical-DH fixture -> ``robot_descriptions / ur5_description``.
  1.46 m position drift vs upstream becomes 0.
- iiwa14: ``kuka_iiwa14_specs()`` -> ``robot_descriptions / iiwa14_description``,
  base ``base`` / ee ``iiwa_link_ee_kuka``.
- Franka Panda: ``franka_panda_specs()`` -> ``robot_descriptions / panda_description``,
  base ``panda_link0`` / ee ``panda_link8``.
- YAM: re-vendored from ``robot_descriptions / yam_description``
  (the v1.2 revision had drifted 285 mm from upstream).
- PiPER: re-vendored from ``robot_descriptions / piper_description``
  (the v1.2 revision had drifted ~10 mm from upstream).

Adds:

- ``fixture_source`` field in MANIFEST schema, REQUIRED for every arm.
  Loader rejects empty. One-line provenance string per arm.
- ``tests/test_prebuilt_fixture_parity.py``: parametrised regression
  test that asserts ``module.fk(q) == upstream.fk(q)`` at machine
  precision on every arm whose source is reachable via
  ``robot_descriptions`` (9 arms covered; 11/11 pass).
- README "Where each fixture comes from" section with auto-regen'd
  fixture-provenance table from the new manifest field.

Not in scope this PR:

- xArm7: switching its fixture from specs to URDF hangs ``emit_artifact``
  on the manufacturer URDF (>60 s, no error). Reverted xArm7 to its
  specs fixture (audit shows 3.6 µm / 9 µrad drift -- below any robot's
  repeatability). Tracked as #312.
- Gen3: vendored from Kinovarobotics / ros_kortex upstream. The
  ``fixture_source`` line names the original source rather than
  ``robot_descriptions /``, so the parity test doesn't cover it
  automatically. Audit shows perfect match.

Q-vectors returned by UR5 / iiwa14 / Panda / YAM / PiPER differ from
v1.2 because they solve a different chain now (the real manufacturer
chain). This is a v1.3.0 minor bump signaling the behavior shift.
Users with v1.2-specific calibration baked in should pin the v1.2.x
range until they re-calibrate to the manufacturer URDF.

Bench updates per ``examples/04_compare_vs_eaik.py``:
- UR5: 532 µs / FK 2e-9 -> 521 µs / FK 6.3e-12
- iiwa14: 4.54 ms / FK 4e-13 -> 4.83 ms / FK 5.1e-13
- Franka Panda: 29.27 ms / FK 1.0e-6 -> 29.57 ms / FK 1.2e-6
- YAM: 1.03 ms / FK 5.4e-9 -> 1.08 ms / FK 7.6e-9
- PiPER: 1.17 ms / FK 9.0e-6 -> 1.10 ms / FK 9.7e-6

File: tests/fixtures/piper.urdf (robot description, URDF)
Before this commit: robot piper, 8 links, 7 joints
Links:
- removed link dummy_link
- added link gripper_base, mass 0.145318531013916; collision mesh filename=/Users/siddh/.cache/robot_descriptions/Piper_ros/src/piper_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; visual mesh filename=/Users/siddh/.cache/robot_descriptions/Piper_ros/src/piper_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
- added link link7, mass 0.0303534920715906; collision mesh filename=/Users/siddh/.cache/robot_descriptions/Piper_ros/src/piper_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; visual mesh filename=/Users/siddh/.cache/robot_descriptions/Piper_ros/src/piper_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
- added link link8, mass 0.0303534920715904; collision mesh filename=/Users/siddh/.cache/robot_descriptions/Piper_ros/src/piper_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; visual mesh filename=/Users/siddh/.cache/robot_descriptions/Piper_ros/src/piper_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
- link base_link: mass 1.02 -> 0.333893486740112; geometry collision mesh filename=/Users/siddh/.cache/robot_descriptions/Piper_ros/src/piper_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; visual mesh filename=/Users/siddh/.cache/robot_descriptions/Piper_ros/src/piper_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
- link link1: mass 0.71 -> 0.215052383265765; geometry collision mesh filename=/Users/siddh/.cache/robot_descriptions/Piper_ros/src/piper_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; visual mesh filename=/Users/siddh/.cache/robot_descriptions/Piper_ros/src/piper_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
- link link2: mass 1.17 -> 0.463914239236335; geometry collision mesh filename=/Users/siddh/.cache/robot_descriptions/Piper_ros/src/piper_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; visual mesh filename=/Users/siddh/.cache/robot_descriptions/Piper_ros/src/piper_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
- link link3: mass 0.5 -> 0.219942452993132; geometry collision mesh filename=/Users/siddh/.cache/robot_descriptions/Piper_ros/src/piper_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; visual mesh filename=/Users/siddh/.cache/robot_descriptions/Piper_ros/src/piper_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
- link link4: mass 0.38 -> 0.131814339939458; geometry collision mesh filename=/Users/siddh/.cache/robot_descriptions/Piper_ros/src/piper_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; visual mesh filename=/Users/siddh/.cache/robot_descriptions/Piper_ros/src/piper_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
- link link5: mass 0.383 -> 0.134101341225523; geometry collision mesh filename=/Users/siddh/.cache/robot_descriptions/Piper_ros/src/piper_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; visual mesh filename=/Users/siddh/.cache/robot_descriptions/Piper_ros/src/piper_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
- link link6: mass 0.007 -> 0.00699089613564366; geometry collision mesh filename=/Users/siddh/.cache/robot_descriptions/Piper_ros/src/piper_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; visual mesh filename=/Users/siddh/.cache/robot_descriptions/Piper_ros/src/piper_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
Joints:
- removed joint base_to_dummy
- added joint joint6_to_gripper_base: type fixed, parent link6, child gripper_base, origin xyz=0.0 0.0 0.0 rpy=0.0 -0.0 0.0, axis 1.0 0.0 0.0
- added joint joint7: type prismatic, parent gripper_base, child link7, origin xyz=0.0 0.0 0.1358 rpy=1.5708 -0.0 0.0, axis 0.0 0.0 1.0, limit lower=0.0 upper=0.035 effort=10.0 velocity=1.0
- added joint joint8: type prismatic, parent gripper_base, child link8, origin xyz=0.0 0.0 0.1358 rpy=1.5708 -0.0 3.1415853071795867, axis 0.0 0.0 -1.0, limit lower=-0.035 upper=0.0 effort=10.0 velocity=1.0
- joint joint1: axis 0 0 1 -> 0.0 0.0 1.0; limit lower=-2.618 upper=2.168 effort=100 velocity=5 -> lower=-2.618 upper=2.168 effort=100.0 velocity=5.0; origin xyz=0 0 0.123 rpy=0 0 0 -> xyz=0.0 0.0 0.123 rpy=0.0 -0.0 0.0
- joint joint2: axis 0 0 1 -> 0.0 0.0 1.0; limit lower=0 upper=3.14 effort=100 velocity=5 -> lower=0.0 upper=3.14 effort=100.0 velocity=5.0; origin xyz=0 0 0 rpy=1.5708 -0.1359 -3.1416 -> xyz=0.0 0.0 0.0 rpy=1.5708 -0.10094999999999998 3.1415853071795867
- joint joint3: axis 0 0 1 -> 0.0 0.0 1.0; limit lower=-2.967 upper=0 effort=100 velocity=5 -> lower=-2.967 upper=0.0 effort=100.0 velocity=5.0; origin xyz=0.28503 0 0 rpy=0 0 -1.7939 -> xyz=0.28503 0.0 0.0 rpy=0.0 -0.0 -1.759
- joint joint4: axis 0 0 1 -> 0.0 0.0 1.0; limit lower=-1.745 upper=1.745 effort=100 velocity=5 -> lower=-1.745 upper=1.745 effort=100.0 velocity=5.0; origin xyz=-0.021984 -0.25075 0 rpy=1.5708 0 0 -> xyz=-0.021984 -0.25075 0.0 rpy=1.5708 -0.0 0.0
- joint joint5: axis 0 0 1 -> 0.0 0.0 1.0; limit lower=-1.22 upper=1.22 effort=100 velocity=5 -> lower=-1.22 upper=1.22 effort=100.0 velocity=5.0; origin xyz=0 0 0 rpy=-1.5708 0 0 -> xyz=0.0 0.0 0.0 rpy=-1.5708 -0.0 0.0
- joint joint6: axis 0 0 1 -> 0.0 0.0 1.0; limit lower=-2.0944 upper=2.0944 effort=100 velocity=3 -> lower=-2.0944 upper=2.0944 effort=100.0 velocity=3.0; origin xyz=8.8259E-05 -0.091 0 rpy=1.5708 0 0 -> xyz=8.8259e-05 -0.091 0.0 rpy=1.5708 -0.0 0.0

File: tests/fixtures/ur5.urdf (robot description, URDF)
Before this commit: robot ur5, 8 links, 7 joints
Links:
- added link base, mass 0.0
- added link tool0, mass 0.0
- added link world
- link base_link: mass None -> 4.0; geometry collision mesh filename=/Users/siddh/.cache/robot_descriptions/example-robot-data/r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; visual mesh filename=/Users/siddh/.cache/robot_descriptions/example-robot-data/r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
- link ee_link: mass None -> 0.0; geometry collision box size=0.01 0.01 0.01
- link forearm_link: mass None -> 2.275; geometry collision mesh filename=/Users/siddh/.cache/robot_descriptions/example-robot-data/r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; visual mesh filename=/Users/siddh/.cache/robot_descriptions/example-robot-data/r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
- link shoulder_link: mass None -> 3.7; geometry collision mesh filename=/Users/siddh/.cache/robot_descriptions/example-robot-data/r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; visual mesh filename=/Users/siddh/.cache/robot_descriptions/example-robot-data/r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
- link upper_arm_link: mass None -> 8.393; geometry collision mesh filename=/Users/siddh/.cache/robot_descriptions/example-robot-data/r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; visual mesh filename=/Users/siddh/.cache/robot_descriptions/example-robot-data/r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
- link wrist_1_link: mass None -> 1.219; geometry collision mesh filename=/Users/siddh/.cache/robot_descriptions/example-robot-data/r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; visual mesh filename=/Users/siddh/.cache/robot_descriptions/example-robot-data/r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
- link wrist_2_link: mass None -> 1.219; geometry collision mesh filename=/Users/siddh/.cache/robot_descriptions/example-robot-data/r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; visual mesh filename=/Users/siddh/.cache/robot_descriptions/example-robot-data/r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
- link wrist_3_link: mass None -> 0.1879; geometry collision mesh filename=/Users/siddh/.cache/robot_descriptions/example-robot-data/r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; visual mesh filename=/Users/siddh/.cache/robot_descriptions/example-robot-data/r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
Joints:
- added joint base_link-base_fixed_joint: type fixed, parent base_link, child base, origin xyz=0.0 0.0 0.0 rpy=0.0 -0.0 3.1415926535895866, axis 1.0 0.0 0.0
- added joint world_joint: type fixed, parent world, child base_link, origin xyz=0.0 0.0 0.0 rpy=0.0 -0.0 0.0, axis 1.0 0.0 0.0
- added joint wrist_3_link-tool0_fixed_joint: type fixed, parent wrist_3_link, child tool0, origin xyz=0.0 0.0823 0.0 rpy=-1.57079632679 -0.0 0.0, axis 1.0 0.0 0.0
- joint ee_fixed_joint: axis (none) -> 1.0 0.0 0.0; origin xyz=0 0 0.0823 rpy=0 0 0 -> xyz=0.0 0.0823 0.0 rpy=0.0 -0.0 1.57079632679
- joint elbow_joint: axis 0 0 1 -> 0.0 1.0 0.0; limit lower=-3.14159265358979 upper=3.14159265358979 effort=150 velocity=3.15 -> lower=-3.14159265359 upper=3.14159265359 effort=150.0 velocity=3.15; origin xyz=-0.425 0 0 rpy=0 0 0 -> xyz=0.0 -0.1197 0.425 rpy=0.0 -0.0 0.0
- joint shoulder_lift_joint: axis 0 0 1 -> 0.0 1.0 0.0; limit lower=-6.28318530717959 upper=6.28318530717959 effort=150 velocity=3.15 -> lower=-6.28318530718 upper=6.28318530718 effort=150.0 velocity=3.15; origin xyz=0 0 0.089159 rpy=1.5707963267948966 0 0 -> xyz=0.0 0.13585 0.0 rpy=0.0 1.57079632679 0.0
- joint shoulder_pan_joint: axis 0 0 1 -> 0.0 0.0 1.0; limit lower=-6.28318530717959 upper=6.28318530717959 effort=150 velocity=3.15 -> lower=-6.28318530718 upper=6.28318530718 effort=150.0 velocity=3.15; origin xyz=0 0 0 rpy=0 0 0 -> xyz=0.0 0.0 0.089159 rpy=0.0 -0.0 0.0
- joint wrist_1_joint: axis 0 0 1 -> 0.0 1.0 0.0; limit lower=-6.28318530717959 upper=6.28318530717959 effort=28 velocity=3.2 -> lower=-6.28318530718 upper=6.28318530718 effort=28.0 velocity=3.2; origin xyz=-0.39225 0 0 rpy=0 0 0 -> xyz=0.0 0.0 0.39225 rpy=0.0 1.57079632679 0.0
- joint wrist_2_joint: axis 0 0 1 -> 0.0 0.0 1.0; limit lower=-6.28318530717959 upper=6.28318530717959 effort=28 velocity=3.2 -> lower=-6.28318530718 upper=6.28318530718 effort=28.0 velocity=3.2; origin xyz=0 0 0.10915 rpy=1.5707963267948966 0 0 -> xyz=0.0 0.093 0.0 rpy=0.0 -0.0 0.0
- joint wrist_3_joint: axis 0 0 1 -> 0.0 1.0 0.0; limit lower=-6.28318530717959 upper=6.28318530717959 effort=28 velocity=3.2 -> lower=-6.28318530718 upper=6.28318530718 effort=28.0 velocity=3.2; origin xyz=0 0 0.09465 rpy=-1.5707963267948966 0 0 -> xyz=0.0 0.0 0.09465 rpy=0.0 -0.0 0.0

File: tests/fixtures/yam.urdf (robot description, URDF)
Before this commit: robot yam_v0, 7 links, 6 joints
Joints:
- joint joint1: axis 0 0 1 -> 0.0 0.0 1.0; limit lower=-2.61799 upper=3.13 effort=10 velocity=10 -> lower=-2.61799 upper=3.13 effort=10.0 velocity=10.0; origin xyz=-3.55271e-18 -1.05495e-18 0.0631 rpy=0 -0 1.5708 -> xyz=-3.55271e-18 -1.05495e-18 0.0631 rpy=0.0 -0.0 1.5708
- joint joint2: axis 0 0 1 -> 0.0 0.0 1.0; limit lower=0 upper=3.65 effort=10 velocity=10 -> lower=0.0 upper=3.65 effort=10.0 velocity=10.0; origin xyz=2.5e-05 -0.02 0.0409 rpy=1.5708 -1.98004e-28 1.5708 -> xyz=2.5e-05 -0.02 0.0409 rpy=1.5708 -1.9800400000000002e-28 1.5708
- joint joint3: axis 0 0 1 -> 0.0 0.0 1.0; limit lower=0 upper=3.13 effort=10 velocity=10 -> lower=0.0 upper=3.13 effort=10.0 velocity=10.0; origin xyz=0.264 0 6.77626e-21 rpy=-3.14159 1.26218e-29 7.88861e-31 -> xyz=0.264 0.0 6.77626e-21 rpy=-3.14159 1.26218e-29 7.88861e-31
- joint joint4: axis 0 0 1 -> 0.0 0.0 1.0; limit lower=-1.5708 upper=1.5708 effort=10 velocity=10 -> lower=-1.5708 upper=1.5708 effort=10.0 velocity=10.0
- joint joint5: axis 0 0 1 -> 0.0 0.0 1.0; limit lower=-1.5708 upper=1.5708 effort=10 velocity=10 -> lower=-1.5708 upper=1.5708 effort=10.0 velocity=10.0; origin xyz=-0.0739968 -0.0395003 2.44738e-05 rpy=-1.5708 1.5708 0 -> xyz=-0.0739968 -0.0395003 2.44738e-05 rpy=1.5707926535897934 1.5707926535897934 3.141592653589793
- joint joint6: axis 0 0 1 -> 0.0 0.0 1.0; limit lower=-2.0944 upper=2.0944 effort=10 velocity=10 -> lower=-2.0944 upper=2.0944 effort=10.0 velocity=10.0
